File: pcb/right_kicad/bifrost_right_thumb.kicad_pcb (KiCad board)
At the start: 2 copper layers, 43 x 32.8 mm, 4 parts, among them SW44 UNASSIGNED_44, SW45 UNASSIGNED_45

Commit message: Update PCB designs
Parts:
- added C1: 100n, Capacitor_SMD:C_0402_1005Metric, B.Cu at (120.0, 105.4)
- added C2: 100n, Capacitor_SMD:C_0402_1005Metric, B.Cu at (138.9, 104.4)
- added D1: WS2812B-2020, LED_SMD:LED_WS2812B-2020_PLCC4_2.0x2.0mm, F.Cu at (120.7, 105.3)
- added D2: WS2812B-2020, LED_SMD:LED_WS2812B-2020_PLCC4_2.0x2.0mm, F.Cu at (139.6, 104.4)
- added J1: Conn_01x05, Connector_PinHeader_1.27mm:PinHeader_1x05_P1.27mm_Vertical, B.Cu at (136.4, 90.1)
- SW1: renamed from SW44; value UNASSIGNED_44 -> 1U
- SW2: renamed from SW45; value UNASSIGNED_45 -> 1U
- moved H2 243.8 mm to (148.6, 99.5), turned to 157.5 degrees
- moved SW2 242.8 mm to (138.9, 99.2), turned to 0 degrees
- moved H1 241.6 mm to (129.2, 99.5), turned to 157.5 degrees
- moved SW1 240.2 mm to (119.5, 100.3), turned to 6.179 degrees
Connections:
- SW1 pad 1: unconnected-(SW44-Pad1) -> PIN_T1
- SW2 pad 1: unconnected-(SW45-Pad1) -> PIN_T2
Routing:
- net RGB_PWR: track 0.00 -> 53.9 mm, vias 0 -> 2
- net RGB: track 0.00 -> 28.4 mm
- net PIN_T1: track 0.00 -> 17.7 mm
- net Net-(D1-DOUT): track 0.00 -> 17.5 mm
- net PIN_T2: track 0.00 -> 5.15 mm
- added copper zone on B.Cu, net GND
- added copper zone on F.Cu, net GND
Other:
- board size 43 x 32.8 mm -> 44.8 x 20.8 mm
