File: pcb/right_kicad/bifrost_right.kicad_pcb (KiCad board)
At the start: 2 copper layers, 142.9 x 80.3 mm, 65 parts, among them J1 HRO_TYPE-C-31-M-12, J2 Conn_01x02, J3 Conn_01x06, J4 Conn_01x05, Q1 AO3401A, Q2 2N7002, Q3 AO3401A, SW1 1U, SW10 1U, SW11 1U, SW12 1U, SW13 1U, SW14 1U, SW15 1U, SW16 1U, SW17 1U, SW18 2.25U, SW19 1U, SW2 1U, SW20 1U, SW21 1.5U, SW22 1U, SW23 1U, SW3 1U, SW4 1U, SW5 1U, SW6 1U, SW7 1U, SW8 1U, SW9 1U, T1 TS24CA, U1 MDBT50Q-1MV2, U2 TP4057, U3 SRV05-4, X1 32.768kHz

Commit message: Update PCB layouts and production files
Parts:
- added G***: LOGO, Smidr:Logo, F.Cu at (184.2, 89.7)
- added G***: LOGO, Smidr:Logo, B.Cu at (184.2, 89.7)
Other:
- board text added: "rev.0.1"
- board text removed: "Bifrǫst v0.1"

Commit message: Update PCB BOM and manufacturing outputs
Parts:
- removed C10: 10u, Capacitor_SMD:C_0402_1005Metric
- removed the R7 at (167.1, 58.3)
- C6: renamed from C4; value 0.1u -> 100n
- C8: value 0.1u -> 100n
- L1: footprint Inductor_SMD:L_0402_1005Metric -> Inductor_SMD:L_0603_1608Metric
- R7: renamed from R6; value 4k -> 3.3k
- R8: renamed from R9; value 100R -> 100
- moved C1 0.10 mm to (77.7, 107.7)
- moved C3 0.10 mm to (81.1, 107.7)
- renumbered C5 to C4, C6 to C5, R11 to R10, R8 to R4, R4 to R5, R5 to R6, R10 to R9
Connections:
- net CS renamed nCS
Routing:
- net +5V: track 129.0 -> 126.4 mm
- net Net-(C10-Pad1): track 1.60 -> 0.00 mm
- net GND: vias 902 -> 903

Commit message: Refactor application implementation
Parts:
- U2: footprint Package_TO_SOT_SMD:TSOT-23-6 -> Package_TO_SOT_SMD:SOT-23-6
Routing:
- net GND: track 20.6 -> 21.7 mm

Commit message: Update Bifrost case and PCB outputs
Parts:
- added TP1: SWDIO, TestPoint:TestPoint_THTPad_D1.0mm_Drill0.5mm, B.Cu at (83.2, 118.1)
- added TP2: SWDCLK, TestPoint:TestPoint_THTPad_D1.0mm_Drill0.5mm, B.Cu at (84.8, 118.1)
Connections:
- J4 pad 2: RGB -> GND
- J4 pad 3: GND -> RGB
- U1 pad 51: unconnected-(U1-SWDIO-Pad51) -> Net-(U1-SWDIO)
- U1 pad 53: unconnected-(U1-SWDCLK-Pad53) -> Net-(U1-SWDCLK)
Routing:
- net Net-(U1-SWDCLK): track 0.00 -> 4.92 mm
- net Net-(U1-SWDIO): track 0.00 -> 2.99 mm
- net RGB: track 33.3 -> 34.6 mm
- net GND: vias 903 -> 901
