File: pcb/right_kicad/bifrost_right.kicad_pcb (KiCad board)
At the start: 2 copper layers, 142.9 x 80.3 mm, 67 parts, among them J1 HRO_TYPE-C-31-M-12, J2 Conn_01x02, J3 Conn_01x06, J4 Conn_01x05, Q1 AO3401A, Q2 2N7002, Q3 AO3401A, SW1 1U, SW10 1U, SW11 1U, SW12 1U, SW13 1U, SW14 1U, SW15 1U, SW16 1U, SW17 1U, SW18 2.25U, SW19 1U, SW2 1U, SW20 1U, SW21 1.5U, SW22 1U, SW23 1U, SW3 1U, SW4 1U, SW5 1U, SW6 1U, SW7 1U, SW8 1U, SW9 1U, T1 TS24CA, U1 MDBT50Q-1MV2, U2 TP4057, U3 SRV05-4, X1 32.768kHz

Commit message: Update PCB plate and stabilizer designs
Routing:
- net GND: vias 901 -> 898

Commit message: Update PCB circuits and manufacturing data
Parts:
- removed the C8 at (190.9, 53.0)
- removed the D1 at (170.7, 52.5)
- R6: renamed from R3; value 1.5k -> 1k
- renumbered C9 to C8, D2 to D1, J3 to J1, J1 to J2, J2 to J3, L3 to L2, L2 to L3, Q3 to Q1, Q1 to Q3, R5 to R1, R4 to R10, R6 to R2, R1 to R3, R2 to R4, R10 to R5, SW8 to SW10, SW14 to SW12, SW18 to SW13, SW3 to SW14, SW6 to SW15, SW9 to SW16, SW12 to SW17, SW15 to SW18, SW4 to SW2, SW22 to SW20, SW16 to SW21, SW20 to SW22, SW7 to SW3, SW10 to SW4, SW13 to SW5, SW17 to SW6, SW21 to SW7, SW2 to SW8, SW5 to SW9, U3 to U1, U1 to U2, U2 to U3
Connections:
- J2 pad A1: Earth -> GND
- J2 pad A12: Earth -> GND
- J2 pad B1: Earth -> GND
- J2 pad B12: Earth -> GND
- J2 pad SH: Earth -> Net-(J2-SHIELD)
- L3 pad 1: Earth -> Net-(J2-SHIELD)
Routing:
- net Earth: track 14.1 -> 0.00 mm
- net Net-(J2-SHIELD): track 0.00 -> 3.12 mm
- net GND: vias 898 -> 900
Other:
- board text added: "rev.0.2"
- board text removed: "rev.0.1"
