File: pcb/right_kicad/bifrost_right_trackball.kicad_pcb (KiCad board)
At the start: 2 copper layers, 18.6 x 20.2 mm, 12 parts, among them J1 Conn_01x06, U1 PMW3610, U2 MCP1700x-180xxTT

Commit message: Update trackball PCB and case
Parts:
- moved J1 0.51 mm to (146.8, 102.9)
Routing:
- net GND: vias 2 -> 9
Changed lines of the file:
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@@
 	(footprint "Connector_PinHeader_1.27mm:PinHeader_1x06_P1.27mm_Vertical"
 		(layer "B.Cu")
-		(at 146.8 102.398751)
+		(at 146.8 102.9038)
 		(descr "Through hole straight pin header, 1x06, 1.27mm pitch, single row")
 		(tags "Through hole pin header THT 1x06 1.27mm single row")
@@
 	)
 	(via
+		(at 135.90625 86.41875)
+		(size 0.4)
+		(drill 0.2)
+		(layers "F.Cu" "B.Cu")
+		(free yes)
+		(net "GND")
+	)
+	(via
 		(at 130.70625 102.81875)
 		(size 0.4)
@@
 	)
 	(via
+		(at 131.30625 88.41875)
+		(size 0.4)
+		(drill 0.2)
+		(layers "F.Cu" "B.Cu")
+		(free yes)
+		(net "GND")
+	)
+	(via
+		(at 130.90625 91.41875)
+		(size 0.4)
+		(drill 0.2)
+		(layers "F.Cu" "B.Cu")
+		(free yes)
+		(net "GND")
+	)
+	(via
+		(at 141.90625 86.41875)
+		(size 0.4)
+		(drill 0.2)
+		(layers "F.Cu" "B.Cu")
+		(free yes)
+		(net "GND")
+	)
+	(via
+		(at 143.70625 104.81875)
+		(size 0.4)
+		(drill 0.2)
+		(layers "F.Cu" "B.Cu")
+		(free yes)
+		(net "GND")
+	)
+	(via
 		(at 130.10625 92.61875)
 		(size 0.4)
@@
 		(net "GND")
 	)
+	(via
+		(at 146.90625 91.01875)
+		(size 0.4)
+		(drill 0.2)
+		(layers "F.Cu" "B.Cu")
+		(free yes)
+		(net "GND")
+	)
+	(via
+		(at 147.70625 104.81875)
+		(size 0.4)
+		(drill 0.2)
+		(layers "F.Cu" "B.Cu")
+		(free yes)
+		(net "GND")
+	)
 	(segment
 		(start 132.50625 104.00625)
@@
 	)
 	(segment
+		(start 147.559803 102.058947)
+		(end 146.8 102.81875)
+		(width 0.3)
+		(layer "B.Cu")
+		(net "+3V3")
+	)
+	(segment
+		(start 147.052697 95.365197)
+		(end 147.559803 95.872303)
+		(width 0.3)
+		(layer "B.Cu")
+		(net "+3V3")
+	)
+	(segment
 		(start 130.10625 89.01875)
 		(end 130.10625 91.411643)
@@
 	)
 	(segment
-		(start 147.052697 94.965197)
-		(end 147.559803 95.472303)
-		(width 0.3)
-		(layer "B.Cu")
-		(net "+3V3")
-	)
-	(segment
 		(start 146.90625 92.01875)
-		(end 146.90625 94.611643)
-		(width 0.3)
-		(layer "B.Cu")
-		(net "+3V3")
-	)
-	(segment
-		(start 147.559803 101.638948)
-		(end 146.8 102.398751)
+		(end 146.90625 95.011643)
 		(width 0.3)
 		(layer "B.Cu")
@@
 	)
 	(segment
-		(start 147.70625 95.825857)
-		(end 147.70625 101.285394)
-		(width 0.3)
-		(layer "B.Cu")
-		(net "+3V3")
-	)
-	(segment
 		(start 147.70625 91.011643)
 		(end 147.70625 89.01875)
@@
 		(start 146.90625 92.01875)
 		(end 147.559803 91.365197)
+		(width 0.3)
+		(layer "B.Cu")
+		(net "+3V3")
+	)
+	(segment
+		(start 147.70625 96.225857)
+		(end 147.70625 101.705393)
 		(width 0.3)
 		(layer "B.Cu")
@@
 	)
 	(arc
-		(start 147.70625 101.285394)
-		(mid 147.66819 101.476736)
-		(end 147.559803 101.638948)
-		(width 0.3)
-		(layer "B.Cu")
-		(net "+3V3")
-	)
-	(arc
 		(start 130.252697 91.765197)
 		(mid 130.14431 91.602985)
@@
 	)
 	(arc
+		(start 147.70625 96.225857)
+		(mid 147.66819 96.034515)
+		(end 147.559803 95.872303)
+		(width 0.3)
+		(layer "B.Cu")
+		(net "+3V3")
+	)
+	(arc
 		(start 130.10625 89.01875)
 		(mid 131.131376 86.543876)
@@
 	)
 	(arc
-		(start 147.052697 94.965197)
-		(mid 146.94431 94.802985)
-		(end 146.90625 94.611643)
-		(width 0.3)
-		(layer "B.Cu")
-		(net "+3V3")
-	)
-	(arc
-		(start 147.70625 95.825857)
-		(mid 147.66819 95.634515)
-		(end 147.559803 95.472303)
+		(start 147.052697 95.365197)
+		(mid 146.94431 95.202985)
+		(end 146.90625 95.011643)
 		(width 0.3)
 		(layer "B.Cu")
@@
 		(net "+3V3")
 	)
+	(arc
+		(start 147.70625 101.705393)
+		(mid 147.66819 101.896735)
+		(end 147.559803 102.058947)
+		(width 0.3)
+		(layer "B.Cu")
+		(net "+3V3")
+	)
 	(segment
 		(start 131.70625 94.89875)
@@
 	)
 	(segment
-		(start 144.25625 102.398751)
-		(end 145.159803 101.495198)
-		(width 0.3)
-		(layer "B.Cu")
-		(net "Net-(U1-+VCSEL)")
-	)
-	(segment
-		(start 132.50625 89.01875)
-		(end 132.50625 89.571643)
-		(width 0.3)
-		(layer "B.Cu")
-		(net "Net-(U1-+VCSEL)")
-	)
-	(segment
-		(start 145.452697 95.472303)
-		(end 145.959803 94.965197)
-		(width 0.3)
-		(layer "B.Cu")
-		(net "Net-(U1-+VCSEL)")
-	)
-	(segment
-		(start 145.30625 101.141644)
-		(end 145.30625 95.825857)
-		(width 0.3)
-		(layer "B.Cu")
-		(net "Net-(U1-+VCSEL)")
-	)
-	(segment
-		(start 144.30625 87.21875)
-		(end 134.30625 87.21875)
-		(width 0.3)
-		(layer "B.Cu")
-		(net "Net-(U1-+VCSEL)")
-	)
-	(segment
-		(start 132.652697 89.925197)
-		(end 133.55625 90.82875)
-		(width 0.3)
-		(layer "B.Cu")
-		(net "Net-(U1-+VCSEL)")
-	)
-	(segment
-		(start 146.10625 94.611643)
-		(end 146.10625 89.01875)
-		(width 0.3)
-		(layer "B.Cu")
-		(net "Net-(U1-+VCSEL)")
-	)
-	(arc
-		(start 145.452697 95.472303)
-		(mid 145.34431 95.634515)
-		(end 145.30625 95.825857)
-		(width 0.3)
-		(layer "B.Cu")
-		(net "Net-(U1-+VCSEL)")
-	)
-	(arc
+		(start 132.50625 89.571643)
+		(end 132.50625 89.01875)
+		(width 0.3)
+		(layer "B.Cu")
+		(net "Net-(U1-+VCSEL)")
+	)
+	(segment
+		(start 133.55625 90.82875)
+		(end 132.652697 89.925197)
+		(width 0.3)
+		(layer "B.Cu")
+		(net "Net-(U1-+VCSEL)")
+	)
+	(segment
+		(start 145.959803 95.365197)
+		(end 145.452697 95.872303)
+		(width 0.3)
+		(layer "B.Cu")
+		(net "Net-(U1-+VCSEL)")
+	)
+	(segment
 		(start 146.10625 89.01875)
-		(mid 145.579042 87.745958)
+		(end 146.10625 95.011643)
+		(width 0.3)
+		(layer "B.Cu")
+		(net "Net-(U1-+VCSEL)")
+	)
+	(segment
+		(start 134.30625 87.21875)
 		(end 144.30625 87.21875)
 		(width 0.3)
@@
 		(net "Net-(U1-+VCSEL)")
 	)
-	(arc
-		(start 145.959803 94.965197)
-		(mid 146.06819 94.802985)
-		(end 146.10625 94.611643)
-		(width 0.3)
-		(layer "B.Cu")
-		(net "Net-(U1-+VCSEL)")
-	)
-	(arc
-		(start 134.30625 87.21875)
-		(mid 133.033458 87.745958)
-		(end 132.50625 89.01875)
+	(segment
+		(start 145.159803 101.495198)
+		(end 144.25625 102.398751)
+		(width 0.3)
+		(layer "B.Cu")
+		(net "Net-(U1-+VCSEL)")
+	)
+	(segment
+		(start 145.30625 96.225857)
+		(end 145.30625 101.141644)
 		(width 0.3)
 		(layer "B.Cu")
@@
 	)
 	(arc
-		(start 145.159803 101.495198)
+		(start 145.959803 95.365197)
+		(mid 146.06819 95.202985)
+		(end 146.10625 95.011643)
+		(width 0.3)
+		(layer "B.Cu")
+		(net "Net-(U1-+VCSEL)")
+	)
+	(arc
+		(start 132.50625 89.01875)
+		(mid 133.033458 87.745958)
+		(end 134.30625 87.21875)
+		(width 0.3)
+		(layer "B.Cu")
+		(net "Net-(U1-+VCSEL)")
+	)
+	(arc
+		(start 145.30625 96.225857)
+		(mid 145.34431 96.034515)
+		(end 145.452697 95.872303)
+		(width 0.3)
+		(layer "B.Cu")
+		(net "Net-(U1-+VCSEL)")
+	)
+	(arc
+		(start 144.30625 87.21875)
+		(mid 145.579042 87.745958)
+		(end 146.10625 89.01875)
+		(width 0.3)
+		(layer "B.Cu")
+		(net "Net-(U1-+VCSEL)")
+	)
+	(arc
+		(start 145.30625 101.141644)
 		(mid 145.26819 101.332986)
-		(end 145.30625 101.141644)
-		(width 0.3)
-		(layer "B.Cu")
-		(net "Net-(U1-+VCSEL)")
-	)
-	(segment
-		(start 144.869799 100.005201)
+		(end 145.159803 101.495198)
+		(width 0.3)
+		(layer "B.Cu")
+		(net "Net-(U1-+VCSEL)")
+	)
+	(segment
+		(start 146.800001 100.363803)
+		(end 144.511197 100.363803)
+		(width 0.2)
+		(layer "F.Cu")
+		(net "SDIO")
+	)
+	(segment
+		(start 144.511197 100.363803)
 		(end 144.25625 100.61875)
 		(width 0.2)
@@
 	)
 	(segment
-		(start 146.799999 99.858754)
-		(end 145.223353 99.858754)
-		(width 0.2)
-		(layer "F.Cu")
-		(net "SDIO")
-	)
-	(arc
-		(start 144.869799 100.005201)
-		(mid 145.032011 99.896814)
-		(end 145.223353 99.858754)
-		(width 0.2)
-		(layer "F.Cu")
-		(net "SDIO")
-	)
-	(segment
-		(start 144.506249 98.588751)
+		(start 146.800001 99.0938)
+		(end 144.5113 99.0938)
+		(width 0.2)
+		(layer "F.Cu")
+		(net "SCLK")
+	)
+	(segment
+		(start 144.5113 99.0938)
 		(end 144.25625 98.83875)
 		(width 0.2)
@@
 	)
 	(segment
-		(start 146.799999 98.588751)
-		(end 144.506249 98.588751)
-		(width 0.2)
-		(layer "F.Cu")
-		(net "SCLK")
-	)
-	(segment
-		(start 144.759995 95.27875)
+		(start 144.25625 95.280046)
 		(end 144.25625 95.27875)
 		(width 0.2)
@@
 	)
 	(segment
-		(start 146.799996 97.318751)
-		(end 144.759995 95.27875)
+		(start 146.800004 97.8238)
+		(end 144.25625 95.280046)
 		(width 0.2)
 		(layer "F.Cu")
@@
 	)
 	(segment
-		(start 146.799999 96.048751)
-		(end 145.30625 94.555002)
+		(start 145.452697 95.206496)
+		(end 146.800001 96.5538)
 		(width 0.2)
 		(layer "F.Cu")
 		(net "MOTION")
 	)
-	(via
-		(at 145.30625 94.555002)
+	(segment
+		(start 145.30625 94.38875)
+		(end 145.30625 94.852942)
+		(width 0.2)
+		(layer "F.Cu")
+		(net "MOTION")
+	)
+	(via
+		(at 145.30625 94.38875)
 		(size 0.4)
 		(drill 0.2)
@@
 		(net "MOTION")
 	)
+	(arc
+		(start 145.452697 95.206496)
+		(mid 145.34431 95.044284)
+		(end 145.30625 94.852942)
+		(width 0.2)
+		(layer "F.Cu")
+		(net "MOTION")
+	)
 	(segment
 		(start 145.30625 90.988751)
-		(end 145.30625 94.555002)
-		(width 0.2)
-		(layer "B.Cu")
+		(end 145.30625 94.38875)
+		(width 0.2)
+		(layer "B.Cu")

Commit message: Update PCB and case designs
Parts:
- moved C1 56.6 mm to (91.7, 49.6)
- moved C2 56.6 mm to (91.7, 54.4)
- moved C3 56.6 mm to (91.7, 47.2)
- moved C7 56.6 mm to (91.7, 52.0)
- moved C9 56.6 mm to (91.7, 59.6)
- moved J1 56.6 mm to (106.8, 62.9)
- moved U2 56.6 mm to (91.7, 63.2)
- moved C5 56.6 mm to (91.7, 56.8)
- moved C4 56.6 mm to (94.5, 46.4)
- moved U1 56.6 mm to (98.9, 59.2)
- moved C6 56.6 mm to (106.1, 53.2)
- moved R10 56.6 mm to (106.1, 50.8)

Commit message: Update PCB layouts and production files
Other:
- board text added: "Bifrost rev.1.0"

Commit message: Update PCB designs and production files
Parts:
- C9: value 3.3uF/16V -> 4.7uF/10V; footprint Capacitor_SMD:C_0603_1608Metric -> Capacitor_SMD:C_0402_1005Metric
- U2: value MCP1700x-180xxTT -> MCP1700T-1802E/TT
- moved C9 0.40 mm to (91.7, 59.2)
