File: pcb/right_kicad/bifrost_right_trackball.kicad_sch (KiCad schematic)
At the start: 1 part, among them U1 PMW3610

Commit message: Update PCB designs
Parts:
- added C1, C3: 10n, Capacitor_SMD:C_0402_1005Metric, symbol Device:C_Small
- added C2, C5, C6: 100n, Capacitor_SMD:C_0402_1005Metric, symbol Device:C_Small
- added C4: 10u, Capacitor_SMD:C_0402_1005Metric, symbol Device:C_Small
- added C7: 1u, Capacitor_SMD:C_0402_1005Metric, symbol Device:C_Small
- added C9: 3.3uF/16V, Capacitor_SMD:C_0603_1608Metric, symbol Device:C_Small
- added J1: Conn_01x06, Connector_PinHeader_1.27mm:PinHeader_1x06_P1.27mm_Vertical, symbol Connector_Generic:Conn_01x06
- added R10: 10k, Resistor_SMD:R_0402_1005Metric, symbol Device:R_Small
- added U2: MCP1700x-180xxTT, Package_TO_SOT_SMD:SOT-23, symbol Regulator_Linear:MCP1700x-180xxTT
Connections:
- net at U1.1 (+VCSEL): now also U1.10 (PASS_T), C1.2
- net GND: now reaches U1.11 (GND)
- net GND: now also C1.1, C3.1, C4.1, C5.1, C6.1, C7.1, C9.1, J1.2 (Pin_2), U2.1 (GND)
- net at U1.12 (CP): now also C2.2
- net at U1.13 (CN): now also C2.1
- net +1V8: now reaches U1.14 (VDD)
- net +1V8: now also C5.2, C9.2, U2.2 (VO)
- net at U1.15 (XYLASER): now also U1.16 (-VCSEL)
- net SDIO: now reaches U1.2 (SDIO)
- net SDIO: now also J1.3 (Pin_3)
- net SCLK: now reaches U1.3 (SCLK)
- net SCLK: now also J1.4 (Pin_4)
- net nCS: now reaches U1.5 (NCS)
- net nCS: now also J1.5 (Pin_5)
- net +3V3: now reaches U1.6 (VDDIO)
- net +3V3: now also C6.2, C7.2, J1.1 (Pin_1), R10.1, U2.3 (VI)
- net at U1.7 (NRESET): now also R10.2
- net MOTION: now reaches U1.8 (MOTION)
- net MOTION: now also J1.6 (Pin_6)
- net at U1.9 (VCP): now also C3.2, C4.2
Other:
- moved on the sheet: U1

Commit message: Update PCB designs and production files
Parts:
- C1, C3: LCSC (none) -> C15195
- C2, C5, C6: LCSC (none) -> C1525
- C4: LCSC (none) -> C15525
- C7: LCSC (none) -> C52923
- C9: value 3.3uF/16V -> 4.7uF/10V; footprint Capacitor_SMD:C_0603_1608Metric -> Capacitor_SMD:C_0402_1005Metric; LCSC (none) -> C23733
- R10: LCSC (none) -> C25744
- U2: value MCP1700x-180xxTT -> MCP1700T-1802E/TT; LCSC (none) -> C150796
Changed lines of the file:
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@@
 			)
 		)
-		(property "LCSC" ""
+		(property "LCSC" "C25744"
 			(at 114.3 91.44 0)
 			(hide yes)
@@
 			)
 		)
-		(property "Value" "3.3uF/16V"
+		(property "Value" "4.7uF/10V"
 			(at 72.39 92.964 0)
 			(show_name no)
@@
 			)
 		)
-		(property "Footprint" "Capacitor_SMD:C_0603_1608Metric"
+		(property "Footprint" "Capacitor_SMD:C_0402_1005Metric"
 			(at 72.39 91.44 0)
 			(hide yes)
@@
 			)
 		)
+		(property "LCSC" "C23733"
+			(at 72.39 91.44 0)
+			(hide yes)
+			(show_name no)
+			(do_not_autoplace no)
+			(effects
+				(font
+					(size 1.27 1.27)
+				)
+			)
+		)
 		(pin "2"
 		)
@@
 			)
 		)
+		(property "LCSC" "C15525"
+			(at 78.74 124.46 0)
+			(hide yes)
+			(show_name no)
+			(do_not_autoplace no)
+			(effects
+				(font
+					(size 1.27 1.27)
+				)
+			)
+		)
 		(pin "2"
 		)
@@
 		)
 		(property "Description" "Unpolarized capacitor, small symbol"
+			(at 83.82 124.46 0)
+			(hide yes)
+			(show_name no)
+			(do_not_autoplace no)
+			(effects
+				(font
+					(size 1.27 1.27)
+				)
+			)
+		)
+		(property "LCSC" "C15195"
 			(at 83.82 124.46 0)
 			(hide yes)
@@
 			)
 		)
+		(property "LCSC" "C15195"
+			(at 83.82 111.76 0)
+			(hide yes)
+			(show_name no)
+			(do_not_autoplace no)
+			(effects
+				(font
+					(size 1.27 1.27)
+				)
+			)
+		)
 		(pin "2"
 		)
@@
 			)
 		)
+		(property "LCSC" "C52923"
+			(at 52.07 93.98 0)
+			(hide yes)
+			(show_name no)
+			(do_not_autoplace no)
+			(effects
+				(font
+					(size 1.27 1.27)
+				)
+			)
+		)
 		(pin "2"
 		)
@@
 			)
 		)
-		(property "Value" "MCP1700x-180xxTT"
+		(property "Value" "MCP1700T-1802E/TT"
 			(at 62.23 85.09 0)
 			(show_name no)
@@
 			)
 		)
+		(property "LCSC" "C150796"
+			(at 62.23 88.9 0)
+			(hide yes)
+			(show_name no)
+			(do_not_autoplace no)
+			(effects
+				(font
+					(size 1.27 1.27)
+				)
+			)
+		)
 		(pin "3"
 		)
@@
 		)
 		(property "Description" "Unpolarized capacitor, small symbol"
+			(at 121.92 91.44 0)
+			(hide yes)
+			(show_name no)
+			(do_not_autoplace no)
+			(effects
+				(font
+					(size 1.27 1.27)
+				)
+			)
+		)
+		(property "LCSC" "C1525"
 			(at 121.92 91.44 0)
 			(hide yes)
@@
 			)
 		)
+		(property "LCSC" "C1525"
+			(at 83.82 101.6 0)
+			(hide yes)
+			(show_name no)
+			(do_not_autoplace no)
+			(effects
+				(font
+					(size 1.27 1.27)
+				)
+			)
+		)
 		(pin "2"
 		)
@@
 			(at 83.82 91.44 0)
 			(hide yes)
+			(show_name no)
+			(do_not_autoplace no)
+			(effects
+				(font
+					(size 1.27 1.27)
+				)
+			)
+		)
+		(property "LCSC" "C1525"
+			(at 83.82 91.44 0)
+			(hide yes)
