File: pcb/left_kicad/bifrost_left.kicad_pcb (KiCad board)
At the start: 2 copper layers, 142.9 x 80.3 mm, 66 parts, among them J1 HRO_TYPE-C-31-M-12, J2 Conn_01x02, J3 Conn_01x06, Q1 AO3401A, Q2 2N7002, Q3 AO3401A, SW1 1.5U, SW10 1U, SW11 1U, SW12 1.25U, SW13 1U, SW14 1U, SW15 1U, SW16 1U, SW17 1U, SW18 1U, SW19 1U, SW2 1.75U, SW20 1U, SW21 1U, SW3 2U, SW4 1.25U, SW5 1U, SW6 1U, SW7 1U, SW8 1.25U, SW9 1U, T1 TS24CA, U1 MDBT50Q-1MV2, U2 TP4057, U3 SRV05-4, X1 32.768kHz

Commit message: Update PCB layouts and production files
Parts:
- added G***: LOGO, Smidr:Logo, F.Cu at (104.0, 89.7)
- added G***: LOGO, Smidr:Logo, B.Cu at (104.0, 89.7)
Other:
- board text added: "rev.0.1"
- board text removed: "Bifrǫst v0.1"

Commit message: Update PCB BOM and manufacturing outputs
Parts:
- removed C10: 10u, Capacitor_SMD:C_0402_1005Metric
- removed the R8 at (91.7, 58.3)
- C6: renamed from C4; value 0.1u -> 100n
- C8: value 0.1u -> 100n
- L1: footprint Inductor_SMD:L_0402_1005Metric -> Inductor_SMD:L_0603_1608Metric
- R7: value 4k -> 3.3k
- R8: renamed from R9; value 100R -> 100
- moved C1 0.10 mm to (210.4, 89.1)
- moved C3 0.10 mm to (207.0, 89.1)
- renumbered C5 to C4, C6 to C5, D2 to D1, D1 to D2, R11 to R10, R12 to R11, R13 to R12, R14 to R13, R10 to R9
Routing:
- net +5V: track 175.6 -> 172.9 mm
- net Net-(C10-Pad1): track 1.60 -> 0.00 mm
- net GND: track 8.44 -> 8.39 mm, vias 959 -> 961

Commit message: Refactor application implementation
Parts:
- U2: footprint Package_TO_SOT_SMD:TSOT-23-6 -> Package_TO_SOT_SMD:SOT-23-6

Commit message: Update Bifrost case and PCB outputs
Parts:
- added TP1: SWDIO, TestPoint:TestPoint_THTPad_D1.0mm_Drill0.5mm, B.Cu at (203.1, 76.3)
- added TP2: SWDCLK, TestPoint:TestPoint_THTPad_D1.0mm_Drill0.5mm, B.Cu at (204.7, 76.3)
Connections:
- J3 pad 2: RGB -> GND
- J3 pad 3: GND -> RGB
- U1 pad 51: unconnected-(U1-SWDIO-Pad51) -> Net-(U1-SWDIO)
- U1 pad 53: unconnected-(U1-SWDCLK-Pad53) -> Net-(U1-SWDCLK)
Routing:
- net Net-(U1-SWDIO): track 0.00 -> 4.46 mm
- net Net-(U1-SWDCLK): track 0.00 -> 2.55 mm
- net RGB: track 37.7 -> 39.0 mm
- net GND: track 8.39 -> 8.43 mm, vias 961 -> 959
