File: pcb/left_kicad/bifrost_left_plate.kicad_pcb (KiCad board)
At the start: 2 copper layers, 148.4 x 87.2 mm, 92 parts

Commit message: Update PCB plate and stabilizer designs
Changed lines of the file:
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@@
 		(duplicate_pad_numbers_are_jumpers no)
 		(fp_line
-			(start 15 -6.3)
-			(end 15 5.2)
-			(stroke
-				(width 0.1)
-				(type default)
-			)
-			(layer "Edge.Cuts")
-		)
-		(fp_line
-			(start 14.5 5.7)
-			(end 9.5 5.7)
+			(start 15.3 -6.3)
+			(end 15.3 5.2)
+			(stroke
+				(width 0.1)
+				(type default)
+			)
+			(layer "Edge.Cuts")
+		)
+		(fp_line
+			(start 14.8 5.7)
+			(end 9.2 5.7)
 			(stroke
 				(width 0.1)
@@
 		(fp_line
 			(start 13.83303 -6.8)
-			(end 14.5 -6.8)
-			(stroke
-				(width 0.1)
-				(type default)
-			)
-			(layer "Edge.Cuts")
-		)
-		(fp_line
-			(start 9.5 -6.8)
+			(end 14.8 -6.8)
+			(stroke
+				(width 0.1)
+				(type default)
+			)
+			(layer "Edge.Cuts")
+		)
+		(fp_line
+			(start 9.2 -6.8)
 			(end 10.16697 -6.8)
 			(stroke
@@
 		)
 		(fp_line
-			(start 9 5.2)
-			(end 9 2.5)
-			(stroke
-				(width 0.1)
-				(type default)
-			)
-			(layer "Edge.Cuts")
-		)
-		(fp_line
-			(start 9 -3.5)
-			(end 9 -6.3)
-			(stroke
-				(width 0.1)
-				(type default)
-			)
-			(layer "Edge.Cuts")
-		)
-		(fp_line
-			(start 8.5 2)
+			(start 8.7 5.2)
+			(end 8.7 2.5)
+			(stroke
+				(width 0.1)
+				(type default)
+			)
+			(layer "Edge.Cuts")
+		)
+		(fp_line
+			(start 8.7 -3.5)
+			(end 8.7 -6.3)
+			(stroke
+				(width 0.1)
+				(type default)
+			)
+			(layer "Edge.Cuts")
+		)
+		(fp_line
+			(start 8.2 2)
 			(end 7.5 2)
 			(stroke
@@
 		(fp_line
 			(start 7.5 -3)
-			(end 8.5 -3)
+			(end 8.2 -3)
 			(stroke
 				(width 0.1)
@@
 		(fp_line
 			(start -7.5 2)
-			(end -8.5 2)
-			(stroke
-				(width 0.1)
-				(type default)
-			)
-			(layer "Edge.Cuts")
-		)
-		(fp_line
-			(start -8.5 -3)
+			(end -8.2 2)
+			(stroke
+				(width 0.1)
+				(type default)
+			)
+			(layer "Edge.Cuts")
+		)
+		(fp_line
+			(start -8.2 -3)
 			(end -7.5 -3)
 			(stroke
@@
 		)
 		(fp_line
-			(start -9 2.5)
-			(end -9 5.2)
-			(stroke
-				(width 0.1)
-				(type default)
-			)
-			(layer "Edge.Cuts")
-		)
-		(fp_line
-			(start -9 -6.3)
-			(end -9 -3.5)
-			(stroke
-				(width 0.1)
-				(type default)
-			)
-			(layer "Edge.Cuts")
-		)
-		(fp_line
-			(start -9.5 5.7)
-			(end -14.5 5.7)
+			(start -8.7 2.5)
+			(end -8.7 5.2)
+			(stroke
+				(width 0.1)
+				(type default)
+			)
+			(layer "Edge.Cuts")
+		)
+		(fp_line
+			(start -8.7 -6.3)
+			(end -8.7 -3.5)
+			(stroke
+				(width 0.1)
+				(type default)
+			)
+			(layer "Edge.Cuts")
+		)
+		(fp_line
+			(start -9.2 5.7)
+			(end -14.8 5.7)
 			(stroke
 				(width 0.1)
@@
 		(fp_line
 			(start -10.16697 -6.8)
-			(end -9.5 -6.8)
-			(stroke
-				(width 0.1)
-				(type default)
-			)
-			(layer "Edge.Cuts")
-		)
-		(fp_line
-			(start -14.5 -6.8)
+			(end -9.2 -6.8)
+			(stroke
+				(width 0.1)
+				(type default)
+			)
+			(layer "Edge.Cuts")
+		)
+		(fp_line
+			(start -14.8 -6.8)
 			(end -13.83303 -6.8)
 			(stroke
@@
 		)
 		(fp_line
-			(start -15 5.2)
-			(end -15 -6.3)
-			(stroke
-				(width 0.1)
-				(type default)
-			)
-			(layer "Edge.Cuts")
-		)
-		(fp_arc
-			(start 15 5.2)
-			(mid 14.853553 5.553553)
-			(end 14.5 5.7)
-			(stroke
-				(width 0.1)
-				(type default)
-			)
-			(layer "Edge.Cuts")
-		)
-		(fp_arc
-			(start 14.5 -6.8)
-			(mid 14.853553 -6.653553)
-			(end 15 -6.3)
+			(start -15.3 5.2)
+			(end -15.3 -6.3)
+			(stroke
+				(width 0.1)
+				(type default)
+			)
+			(layer "Edge.Cuts")
+		)
+		(fp_arc
+			(start 15.3 5.2)
+			(mid 15.153553 5.553553)
+			(end 14.8 5.7)
+			(stroke
+				(width 0.1)
+				(type default)
+			)
+			(layer "Edge.Cuts")
+		)
+		(fp_arc
+			(start 14.8 -6.8)
+			(mid 15.153553 -6.653553)
+			(end 15.3 -6.3)
 			(stroke
 				(width 0.1)
@@
 		)
 		(fp_arc
-			(start 9.5 5.7)
-			(mid 9.146447 5.553553)
-			(end 9 5.2)
-			(stroke
-				(width 0.1)
-				(type default)
-			)
-			(layer "Edge.Cuts")
-		)
-		(fp_arc
-			(start 9 -3.5)
-			(mid 8.853553 -3.146447)
-			(end 8.5 -3)
-			(stroke
-				(width 0.1)
-				(type default)
-			)
-			(layer "Edge.Cuts")
-		)
-		(fp_arc
-			(start 9 -6.3)
-			(mid 9.146447 -6.653553)
-			(end 9.5 -6.8)
-			(stroke
-				(width 0.1)
-				(type default)
-			)
-			(layer "Edge.Cuts")
-		)
-		(fp_arc
-			(start 8.5 2)
-			(mid 8.853553 2.146447)
-			(end 9 2.5)
+			(start 9.2 5.7)
+			(mid 8.846447 5.553553)
+			(end 8.7 5.2)
+			(stroke
+				(width 0.1)
+				(type default)
+			)
+			(layer "Edge.Cuts")
+		)
+		(fp_arc
+			(start 8.7 -3.5)
+			(mid 8.553553 -3.146447)
+			(end 8.2 -3)
+			(stroke
+				(width 0.1)
+				(type default)
+			)
+			(layer "Edge.Cuts")
+		)
+		(fp_arc
+			(start 8.7 -6.3)
+			(mid 8.846447 -6.653553)
+			(end 9.2 -6.8)
+			(stroke
+				(width 0.1)
+				(type default)
+			)
+			(layer "Edge.Cuts")
+		)
+		(fp_arc
+			(start 8.2 2)
+			(mid 8.553553 2.146447)
+			(end 8.7 2.5)
 			(stroke
 				(width 0.1)
@@
 		)
 		(fp_arc
-			(start -8.5 -3)
-			(mid -8.853553 -3.146447)
-			(end -9 -3.5)
-			(stroke
-				(width 0.1)
-				(type default)
-			)
-			(layer "Edge.Cuts")
-		)
-		(fp_arc
-			(start -9 5.2)
-			(mid -9.146447 5.553553)
-			(end -9.5 5.7)
-			(stroke
-				(width 0.1)
-				(type default)
-			)
-			(layer "Edge.Cuts")
-		)
-		(fp_arc
-			(start -9 2.5)
-			(mid -8.853553 2.146447)
-			(end -8.5 2)
-			(stroke
-				(width 0.1)
-				(type default)
-			)
-			(layer "Edge.Cuts")
-		)
-		(fp_arc
-			(start -9.5 -6.8)
-			(mid -9.146447 -6.653553)
-			(end -9 -6.3)
+			(start -8.2 -3)
+			(mid -8.553553 -3.146447)
+			(end -8.7 -3.5)
+			(stroke
+				(width 0.1)
+				(type default)
+			)
+			(layer "Edge.Cuts")
+		)
+		(fp_arc
+			(start -8.7 5.2)
+			(mid -8.846447 5.553553)
+			(end -9.2 5.7)
+			(stroke
+				(width 0.1)
+				(type default)
+			)
+			(layer "Edge.Cuts")
+		)
+		(fp_arc
+			(start -8.7 2.5)
+			(mid -8.553553 2.146447)
+			(end -8.2 2)
+			(stroke
+				(width 0.1)
+				(type default)
+			)
+			(layer "Edge.Cuts")
+		)
+		(fp_arc
+			(start -9.2 -6.8)
+			(mid -8.846447 -6.653553)
+			(end -8.7 -6.3)
 			(stroke
 				(width 0.1)
@@
 		)
 		(fp_arc
-			(start -14.5 5.7)
-			(mid -14.853553 5.553553)
-			(end -15 5.2)
-			(stroke
-				(width 0.1)
-				(type default)
-			)
-			(layer "Edge.Cuts")
-		)
-		(fp_arc
-			(start -15 -6.3)
-			(mid -14.853553 -6.653553)
-			(end -14.5 -6.8)
-			(stroke
-				(width 0.1)
+			(start -14.8 5.7)
+			(mid -15.153553 5.553553)
+			(end -15.3 5.2)
+			(stroke
+				(width 0.1)
+				(type default)
+			)
+			(layer "Edge.Cuts")
+		)
+		(fp_arc
+			(start -15.3 -6.3)
+			(mid -15.153553 -6.653553)
+			(end -14.8 -6.8)
+			(stroke
+				(width 0.1)
