File: pcb/left_kicad/bifrost_left.kicad_sch (KiCad schematic)
At the start: 65 parts, among them J1 HRO_TYPE-C-31-M-12, J2 Conn_01x02, J3 Conn_01x06, Q1 AO3401A, Q2 2N7002, Q3 AO3401A, SW1 1.5U, SW10 1U, SW11 1U, SW12 1.25U, SW13 1U, SW14 1U, SW15 1U, SW16 1U, SW17 1U, SW18 1U, SW19 1U, SW2 1.75U, SW20 1U, SW21 1U, SW3 2U, SW4 1.25U, SW5 1U, SW6 1U, SW7 1U, SW8 1.25U, SW9 1U, T1 TS24CA, U1 MDBT50Q-1MV2, U2 TP4057, U3 SRV05-4, X1 32.768kHz

Commit message: Update PCB circuits and manufacturing data
Parts:
- removed C8: 100n, Capacitor_SMD:C_0402_1005Metric, symbol Device:C_Small
- removed D1: BSD3C051V, Diode_SMD:D_SOD-323, symbol Device:D_TVS_Small
- L3: renamed from L2; footprint Inductor_SMD:L_0402_1005Metric -> (none); JLCPCB Part # C88970 -> (none)
- renumbered C9 to C8, D3 to D1, L3 to L2, Q3 to Q1, Q1 to Q3, R5 to R1, R7 to R10, R8 to R11, R9 to R12, R4 to R13, R6 to R2, R10 to R3, R11 to R4, R12 to R5, R1 to R6, R2 to R7, R13 to R8, R3 to R9, SW14 to SW10, SW17 to SW11, SW20 to SW12, SW3 to SW13, SW7 to SW14, SW11 to SW15, SW15 to SW16, SW18 to SW17, SW21 to SW18, SW4 to SW19, SW5 to SW2, SW8 to SW20, SW12 to SW21, SW9 to SW3, SW13 to SW4, SW16 to SW5, SW19 to SW6, SW2 to SW7, SW6 to SW8, SW10 to SW9, U3 to U1, U1 to U2, U2 to U3
Connections:
- net GND: now also J1.A1 (GND), J1.A12 (GND), J1.B1 (GND), J1.B12 (GND)
- removed net Earth: J1.A1 (GND), J1.A12 (GND), J1.B1 (GND), J1.B12 (GND), J1.SH (SHIELD), L3.1
- new net: J1.SH (SHIELD), L3.1
Other:
- moved on the sheet: L3
